File: GraphicPlus.kicad_pcb (KiCad board)
At the start: 2 copper layers, 100 x 77.5 mm, 23 parts, among them J1 Apple II Expansion Bus, J2 Printer Connector, U1 74LS00, U10 74LS374, U11 74LS373, U2 74LS279, U3 74LS02, U5 74LS74, U6 74LS00, U7 74LS08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

Commit message: rev 2, PC dongle compatibility
Parts:
- added JP1: ~, Jumper:SolderJumper-2_P1.3mm_Open_RoundedPad1.0x1.5mm, B.Cu at (174.6, 69.9)
- added JP2: ~, Jumper:SolderJumper-2_P1.3mm_Open_RoundedPad1.0x1.5mm, B.Cu at (177.2, 69.9)
- added JP3: ~, Jumper:SolderJumper-2_P1.3mm_Open_RoundedPad1.0x1.5mm, B.Cu at (179.7, 69.9)
- added JP4: ~, Jumper:SolderJumper-2_P1.3mm_Open_RoundedPad1.0x1.5mm, B.Cu at (182.2, 69.9)
Connections:
- J2 pad 2: GND -> Net-(J2-Pin_2)
- J2 pad 4: GND -> Net-(J2-Pin_4)
- J2 pad 6: GND -> Net-(J2-Pin_6)
- J2 pad 8: GND -> Net-(J2-Pin_8)
Routing:
- net Net-(J2-Pin_8): track 0.00 -> 1.88 mm
- net Net-(J2-Pin_6): track 0.00 -> 1.88 mm
- net Net-(J2-Pin_4): track 0.00 -> 1.88 mm
- net Net-(J2-Pin_2): track 0.00 -> 1.88 mm
