File: GraphicPlus.kicad_pcb (KiCad board)
At the start: 2 copper layers, 100 x 77.5 mm, 27 parts, among them J1 Apple II Expansion Bus, J2 Printer Connector, U1 74LS00, U10 74LS374, U11 74LS373, U2 74LS279, U3 74LS02, U5 74LS74, U6 74LS00, U7 74LS08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

Commit message: U2 pin 1 supposed to be GND, not +5
Connections:
- U2 pad 1: +5V -> GND
Changed lines of the file:
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@@
       (stroke (width 0.1) (type solid)) (layer "F.Fab"))
     (pad "1" thru_hole rect (at 0 0) (size 1.6 1.6) (drill 0.8) (layers "*.Cu" "*.Mask")
-      (net 3 "+5V") (pinfunction "~{R}") (pintype "input"))
+      (net 2 "GND") (pinfunction "~{R}") (pintype "input"))
     (pad "2" thru_hole oval (at 0 2.54) (size 1.6 1.6) (drill 0.8) (layers "*.Cu" "*.Mask")
       (net 51 "/~{IOSTB}") (pinfunction "~{S1}") (pintype "input"))

Commit message: force +5 on U9alt pin 26
Connections:
- U9 pad 26: unconnected-(U9-NC-Pad26) -> +5V

Commit message: rev3 fixes
Parts:
- C8: value C -> 100p
Changed lines of the file:
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@@
       (net 81 "/ROMA8") (pinfunction "A8") (pintype "input"))
     (pad "26" thru_hole oval (at 15.24 5.08) (size 1.6 1.6) (drill 0.8) (layers "*.Cu" "*.Mask")
-      (net 3 "+5V") (pinfunction "NC") (pintype "no_connect"))
+      (net 3 "+5V") (pinfunction "NC") (pintype "free"))
     (pad "27" thru_hole oval (at 15.24 2.54) (size 1.6 1.6) (drill 0.8) (layers "*.Cu" "*.Mask")
       (net 3 "+5V") (pinfunction "~{PGM}") (pintype "input"))
@@
         (effects (font (size 1 1) (thickness 0.15)))
     )
-    (fp_text value "C" (at 2.5 0) (layer "F.SilkS")
+    (fp_text value "100p" (at 2.5 0) (layer "F.SilkS")
         (effects (font (size 1 0.762) (thickness 0.15)))
     )
